File: hardware/kicad/LNA_and_antenna.sch (KiCad schematic (older format))
At the start: 0 parts

Commit message: Finished port from Altium to KiCAD
Parts:
- added C? (x4): 10uF, ~, symbol C
- added C? (x3): 100nF, ~, symbol C
- added C? (x2): 14pF, ~, symbol C
- added C?: 1pF, ~, symbol C
- added C?: 0pF, ~, symbol C
- added L? (x3): DNP, ~, symbol INDUCTOR
- added L?: 120 ohms @ 100 MHz, ~, symbol INDUCTOR
- added L? (x2): 0.004uH, ~, symbol INDUCTOR
- added L?: 0.07uH, ~, symbol INDUCTOR
- added L?: 0nH, ~, symbol INDUCTOR
- added R?: 68k, ~, symbol R
- added R?: 15k, ~, symbol R
- added U?: PSA4-5043+, symbol PSA4-5043+
- added U?: ADG918, symbol ADG918
- added U?: SMA, symbol SMA
Connections:
- new net: C?.2, L?.1, L?.1, U?.1 (RF_OUT)
- new net: C?.1, U?.3 (RF_IN)
- new net: C?.1, C?.1, R?.1, R?.2, U?.1 (VDD)
- new net: U?.1 (SIG), U?.4 (RFC)
- new net: L?.1, L?.1, L?.2, U?.5 (RF2)
- new net: C?.2, U?.8 (RF1)
- new net: C?.2, C?.2, R?.2
- new net: C?.2, L?.1 (x2)
- new net: C?.1, C?.1, L?.1, L?.2
- new net +3.3V: C?.1, C?.1, C?.1, L?.2, L?.2, R?.1
- new net GND: C?.2, C?.2, C?.2, C?.2, C?.2, L?.2, L?.2, L?.2, L?.2, U?.2 (G), U?.2 (GND), U?.3 (GND), U?.4 (GND), U?.6 (GND), U?.7 (GND)
- new net LNA: C?.1
- new net SWITCH: U?.2 (CTRL)
- new net tx_filter: C?.1, C?.1, L?.1
Other:
- note added: "Note: These caps need to be very low loss (NP0 or ATC)\n"
