File: hardware/kicad/LO.sch (KiCad schematic (older format))
At the start: 0 parts

Commit message: Finished port from Altium to KiCAD
Parts:
- added C? (x2): 1nF, ~, symbol C
- added C?: 10uF, ~, symbol C
- added C? (x9): 10pF, ~, symbol C
- added C?: 16nF, ~, symbol C
- added C?: 500pF, ~, symbol C
- added C? (x8): 0.1uF, ~, symbol C
- added C? (x2): 5pF, ~, symbol C
- added C?: 120pF, ~, symbol C
- added D?: LED, ~, symbol LED
- added L?: 94nH, ~, symbol INDUCTOR
- added L? (x2): 23nH, ~, symbol INDUCTOR
- added R?: 0, ~, symbol R
- added R? (x2): DNP, ~, symbol R
- added R? (x4): 10k, ~, symbol R
- added R?: R, ~, symbol R
- added R?: 23k, ~, symbol R
- added R?: 11k, ~, symbol R
- added R?: 5.1k, ~, symbol R
- added U?: ADF4351, symbol ADF4351
- added U?: FOX924B, symbol FOX924B
Connections:
- new net: C?.1, L?.2, U?.12 (RFoutA+)
- new net: C?.1, L?.2, L?.2, U?.13 (RFoutA-)
- new net: C?.1, C?.1, U?.19 (TEMP)
- new net: C?.1, R?.2, U?.20 (VTune)
- new net: R?.1, U?.22 (RSet)
- new net: C?.1, C?.1, U?.23 (VCOM)
- new net: C?.1, C?.1, U?.24 (VREF)
- new net: R?.1, U?.25 (LD)
- new net: R?.2, R?.2, U?.26 (PDBrf)
- new net: C?.2, U?.29 (REFin)
- new net: R?.2, U?.4 (CE)
- new net: C?.1, C?.1, R?.1, U?.7 (CPout)
- new net: C?.1, U?.3 (OUT)
- new net: D?.1 (A), R?.2
- new net: C?.2, R?.1 (x2)
- new net: C?.1, C?.2, L?.1
- new net +3.3V: C?.1, C?.1, C?.1, C?.1, C?.1, C?.1, C?.1, C?.1, C?.1, C?.1, C?.1, C?.1, L?.1, L?.1, R?.1, R?.1, U?.10 (AVDD), U?.16 (VVCO), U?.17 (VVCO), U?.28 (DVDD), U?.32 (SDVDD), U?.4 (VCC), U?.6 (Vp)
- new net GND: C?.2, C?.2, C?.2, C?.2, C?.2, C?.2, C?.2, C?.2, C?.2, C?.2, C?.2, C?.2, C?.2, C?.2, C?.2, C?.2, C?.2, C?.2, C?.2, C?.2, C?.2, D?.2 (K), R?.1, R?.2, R?.2, R?.2, R?.2, R?.2, R?.2, U?.11 (AGNDVCO), U?.14 (RFoutB+), U?.15 (RFoutB-), U?.18 (AGNDVCO), U?.2 (GND), U?.21 (AGNDVCO), U?.27 (DGND), U?.31 (SDGND), U?.8 (CpGND), U?.9 (AGND)
- new net LE: R?.1, U?.3 (LE)
- new net SCLK: R?.1, U?.1 (CLK)
- new net SI: R?.1, U?.2 (DATA)
Other:
- note added: "10 MHz reference\n"
- note added: "Note: These values were determined experimentally.\nThis terminates the unused output and matches to 50 ohms.\nIt doens't do any filtering."
