File: hardware/kicad/cc430.sch (KiCad schematic (older format))
At the start: 0 parts

Commit message: Finished port from Altium to KiCAD
Parts:
- added C? (x9): 100nF, ~, symbol C
- added C? (x4): 2pF, ~, symbol C
- added C?: 470nF, ~, symbol C
- added C?: DNP, ~, symbol C
- added C?: 0.0022uF, ~, symbol C
- added C? (x2): 27pF, ~, symbol C
- added C? (x4): 10uF, ~, symbol C
- added C?: 100pF, ~, symbol C
- added C? (x5): 0.1uF, ~, symbol C
- added D? (x3): LED, ~, symbol LED
- added P?: CONN_4, symbol CONN_4
- added R? (x3): 330, ~, symbol R
- added R?: 47k, ~, symbol R
- added R?: 56k, 1%, ~, symbol R
- added U?: CC430F5137, symbol CC430F5137
- added U?: 0896BM15A0001, symbol 0896BM15A0001
- added U?: NX3225GA-26MHZ-TI, symbol NX3225GA-26MHZ-TI
Connections:
- new net: R?.2, U?.1 (P2.2)
- new net: R?.2, U?.15 (P3.6)
- new net: R?.2, U?.2 (P2.1)
- new net: C?.1, U?.1 (OUT), U?.25 (RF_XIN)
- new net: C?.1, U?.26 (RF_XOUT), U?.3 (OUT)
- new net: U?.29 (RF_P), U?.4 (BAL)
- new net: U?.3 (BAL), U?.30 (RF_N)
- new net: R?.1, U?.33 (RBIAS)
- new net: P?.1 (P1), U?.39 (TEST)
- new net: C?.2, P?.2 (P2), R?.2, U?.40 (/RST)
- new net: C?.1, C?.1, U?.7 (VCORE)
- new net: C?.1, U?.1 (UNBAL)
- new net: D?.1 (A), R?.1 (x3)
- new net +3.3V: C?.1, C?.1, C?.1, C?.1, C?.1, C?.1, C?.1, C?.1, C?.1, C?.1, C?.1, C?.1, C?.1, C?.1, C?.1, C?.1, C?.1, C?.1, C?.1, C?.1, C?.1, C?.1, P?.4 (P4), R?.1, U?.22 (DVCC), U?.27 (AVCC_RF), U?.28 (AVCC_RF), U?.31 (AVCC_RF), U?.32 (AVCC_RF), U?.34 (GUARD), U?.41 (DVCC), U?.45 (AVCC), U?.8 (DVCC)
- new net CC430_TAP: C?.2
- new net GND: C?.2, C?.2, C?.2, C?.2, C?.2, C?.2, C?.2, C?.2, C?.2, C?.2, C?.2, C?.2, C?.2, C?.2, C?.2, C?.2, C?.2, C?.2, C?.2, C?.2, C?.2, C?.2, C?.2, C?.2, C?.2, C?.2, D?.2 (K), D?.2 (K), D?.2 (K), P?.3 (P3), R?.2, U?.2 (GND), U?.42 (AVSS), U?.49 (VSS), U?.5 (GND), U?.6 (GND)
- new net GPIO0: U?.5 (P1.6)
- new net GPIO1: U?.4 (P1.7)
- new net LE: U?.13 (P1.0)
- new net LE2: U?.11 (P1.2)
- new net SCK: U?.12 (P1.1)
- new net SCK2: U?.10 (P1.3)
- new net SI: U?.6 (P1.5)
- new net SI2: U?.9 (P1.4)
- new net SO2: U?.23 (P2.7)
- new net SWITCH: U?.3 (P2.0)
