File: hardware/kicad/headers.sch (KiCad schematic (older format))
At the start: 11 parts

Commit message: Finished port from Altium to KiCAD
Connections:
- net GPIO2 renamed GPIO0
Changed lines of the file:
@@
 $Descr A4 11693 8268
 encoding utf-8
-Sheet 9 9
+Sheet 8 9
 Title ""
-Date "26 sep 2014"
+Date "27 sep 2014"
 Rev ""
 Comp ""
@@
 GPIO1
 Text HLabel 7050 3500 0    60   BiDi ~ 0
-GPIO2
+GPIO0
 Wire Wire Line
 	7050 3500 7200 3500
