File: hardware/kicad/mixer.sch (KiCad schematic (older format))
At the start: 0 parts

Commit message: Finished port from Altium to KiCAD
Parts:
- added C? (x2): 10pF, ~, symbol C
- added C? (x2): 15pF, ~, symbol C
- added C? (x2): 2.7pF, ~, symbol C
- added L? (x4): 18nH, ~, symbol INDUCTOR
- added L?: 19nH, ~, symbol INDUCTOR
- added U?: ADEX-10L, symbol ADEX-10L
- added U?: B3744, symbol B3744
Connections:
- new net: C?.1, L?.1, L?.2 (x2)
- new net: C?.1, L?.2, U?.2 (IF)
- new net: C?.1, L?.2, U?.6 (LO)
- new net: L?.2, U?.2 (IN)
- new net: L?.1, U?.4 (OUT)
- new net GND: C?.2, C?.2, C?.2, C?.2, C?.2, C?.2, U?.1 (GND), U?.1 (IN_GND), U?.3 (GND), U?.4 (GND), U?.5 (GND), U?.5 (OUT_GND), U?.6 (GND)
- new net LO: C?.1, L?.1
- new net MIX_IN: C?.1, L?.1
- new net MIX_OUT: U?.3 (RF)
