File: hardware/kicad/switch_and_PA.sch (KiCad schematic (older format))
At the start: 0 parts

Commit message: Finished port from Altium to KiCAD
Parts:
- added C? (x2): 10uF, ~, symbol C
- added C? (x5): 100nF, ~, symbol C
- added C?: 14pF, ~, symbol C
- added C?: 0.8pF, ~, symbol C
- added C?: 13.8pF, ~, symbol C
- added C?: 0pF, ~, symbol C
- added L?: 0.004uH, ~, symbol INDUCTOR
- added L?: 0.07uH, ~, symbol INDUCTOR
- added L?: 0.004uF, ~, symbol INDUCTOR
- added L?: 0nH, ~, symbol INDUCTOR
- added L?: 120 ohms @ 100 MHz, ~, symbol INDUCTOR
- added R?: 15k, ~, symbol R
- added R?: 68k, ~, symbol R
- added U?: ADG918, symbol ADG918
- added U?: PSA4-5043+, symbol PSA4-5043+
Connections:
- new net: C?.1, C?.1, R?.1, R?.2, U?.1 (VDD)
- new net: C?.1, U?.5 (RF2)
- new net: C?.1, C?.1, L?.1, U?.8 (RF1)
- new net: C?.2, U?.1 (RF_OUT)
- new net: C?.1, L?.1, U?.3 (RF_IN)
- new net: C?.2, L?.1 (x2)
- new net: C?.1, C?.1, L?.1, L?.2
- new net +3.3V: C?.1, C?.1, C?.1, L?.2, R?.1
- new net GND: C?.2, C?.2, C?.2, C?.2, C?.2, C?.2, C?.2, L?.2, L?.2, R?.2, U?.2 (GND), U?.3 (GND), U?.4 (GND), U?.6 (GND), U?.7 (GND)
- new net LNA: L?.2
- new net MIX_OUT: U?.4 (RFC)
- new net SWITCH: U?.2 (CTRL)
- new net tx_filter: C?.2
Other:
- note added: "Band pass filter for removing stuff above 700 MHz\n"
- note added: "Note: these caps need to be very low loss (NP0 or ATC)\n"
